Commit message: renamed:    interface/config/camera.yaml -> config/camera.yaml 	modified:   interface/franka_description/panda.urdf 	new file:   interface/franka_description/panda_robotiq_arg85.urdf 	new file:   interface/franka_description/panda_robotiq_hande.urdf 	modified:   interface/rerun_interface.py 	deleted:    interface/robotiq_arg85_description/.gitignore 	deleted:    interface/robotiq_arg85_description/.travis.yml 	deleted:    interface/robotiq_arg85_description/README.md 	deleted:    interface/robotiq_arg85_description/images/display.png 	deleted:    interface/robotiq_arg85_description/launch/display.launch 	deleted:    interface/robotiq_arg85_description/package.xml 	deleted:    interface/robotiq_arg85_description/urdf.rviz 	deleted:    interface/robotiq_hande_description/.gitignore 	deleted:    interface/robotiq_hande_description/CMakeLists.txt 	deleted:    interface/robotiq_hande_description/LICENSE 	deleted:    interface/robotiq_hande_description/README.md 	deleted:    interface/robotiq_hande_description/cad_models/coupler.FCStd 	deleted:    interface/robotiq_hande_description/cad_models/coupler.FCStd1 	deleted:    interface/robotiq_hande_description/cad_models/finger.FCStd 	deleted:    interface/robotiq_hande_description/cad_models/finger_collision.FCStd 	deleted:    interface/robotiq_hande_description/cad_models/hande_step.FCStd 	deleted:    interface/robotiq_hande_description/docs/hande_rviz.gif 	deleted:    interface/robotiq_hande_description/meshes/finger.dae 	new file:   interface/robotiq_hande_description/meshes/finger_1.dae 	new file:   interface/robotiq_hande_description/meshes/finger_2.dae 	deleted:    interface/robotiq_hande_description/meshes/finger_collision.dae 	new file:   interface/robotiq_hande_description/meshes/hand-e.dae 	deleted:    interface/robotiq_hande_description/meshes/hande.dae 	deleted:    interface/robotiq_hande_description/package.xml 	modified:   interface/robotiq_hande_description/robotiq_hande.urdf 	deleted:    interface/robotiq_hande_description/rviz/urdf.rviz 	deleted:    interface/robotiq_hande_description/urdf/materials.xacro

File: interface/robotiq_hande_description/robotiq_hande.urdf (robot description, URDF)
Before this commit: robot robotiq_hande, 4 links, 3 joints
Links:
- removed link hande_left_finger
- removed link hande_right_finger
- removed link hande_robotiq_hande_base_link
- removed link world
- added link left_finger, mass 0.03804; collision mesh filename=robotiq_hande_description/meshes/finger_1.dae scale=0.001 0.001 0.001; visual mesh filename=robotiq_hande_description/meshes/finger_1.dae scale=0.001 0.001 0.001
- added link right_finger, mass 0.03804; collision mesh filename=robotiq_hande_description/meshes/finger_2.dae scale=0.001 0.001 0.001; visual mesh filename=robotiq_hande_description/meshes/finger_2.dae scale=0.001 0.001 0.001
- added link robotiq_hande_base_link, mass 0.86387; collision mesh filename=robotiq_hande_description/meshes/hand-e.dae scale=0.001 0.001 0.001; visual mesh filename=robotiq_hande_description/meshes/hand-e.dae scale=0.001 0.001 0.001
- added link robotiq_hande_coupler, mass 0.86387; collision mesh filename=robotiq_hande_description/meshes/coupler.dae scale=0.001 0.001 0.001; visual mesh filename=robotiq_hande_description/meshes/coupler.dae scale=0.001 0.001 0.001
Joints:
- removed joint hande_joint_finger
- removed joint world_to_robotiq_adapter
- added joint joint_finger: type prismatic, parent robotiq_hande_base_link, child left_finger, origin xyz=0 0 0.099 rpy=0 0 0, axis -1 0 0, limit lower=0 upper=0.025 effort=130 velocity=0.15
- added joint robotiq_hande_coupler_to_base: type fixed, parent robotiq_hande_coupler, child robotiq_hande_base_link, origin xyz=0 0 0.0134 rpy=0 0 0
- joint robotiq_hande_base_to_hande_right_finger: child hande_right_finger -> right_finger; mimic joint=hande_joint_finger multiplier=1 offset=0 -> joint=joint_finger multiplier=1 offset=0; parent hande_robotiq_hande_base_link -> robotiq_hande_base_link
