Commit message: modified:   interface/__pycache__/common.cpython-311.pyc 	modified:   interface/__pycache__/rerun_loader_urdf.cpython-311.pyc 	modified:   interface/common.py 	modified:   interface/franka_description/panda.urdf 	modified:   interface/franka_description/panda_arg85.urdf 	modified:   interface/franka_description/panda_hande.urdf 	modified:   interface/franka_description/panda_hande_d435i.urdf 	modified:   interface/interface.py 	modified:   interface/rerun_loader_urdf.py

File: interface/franka_description/panda.urdf (robot description, URDF)
Before this commit: robot panda, 17 links, 16 joints
Links:
- removed link panda_link0
- removed link panda_link0_sc
- removed link panda_link1
- removed link panda_link1_sc
- removed link panda_link2
- removed link panda_link2_sc
- removed link panda_link3
- removed link panda_link3_sc
- removed link panda_link4
- removed link panda_link4_sc
- removed link panda_link5
- removed link panda_link5_sc
- removed link panda_link6
- removed link panda_link6_sc
- removed link panda_link7
- removed link panda_link7_sc
- removed link panda_link8
- added link link0; collision mesh filename=franka_description/meshes/collision/link0.stl; visual mesh filename=franka_description/meshes/visual/link0.dae
- added link link0_sc; collision cylinder length=0.03 radius=0.09; collision sphere radius=0.09
- added link link1; collision mesh filename=franka_description/meshes/collision/link1.stl; visual mesh filename=franka_description/meshes/visual/link1.dae
- added link link1_sc; collision cylinder length=0.283 radius=0.09; collision sphere radius=0.09
- added link link2; collision mesh filename=franka_description/meshes/collision/link2.stl; visual mesh filename=franka_description/meshes/visual/link2.dae
- added link link2_sc; collision cylinder length=0.12 radius=0.09; collision sphere radius=0.09
- added link link3; collision mesh filename=franka_description/meshes/collision/link3.stl; visual mesh filename=franka_description/meshes/visual/link3.dae
- added link link3_sc; collision cylinder length=0.15 radius=0.09; collision sphere radius=0.09
- added link link4; collision mesh filename=franka_description/meshes/collision/link4.stl; visual mesh filename=franka_description/meshes/visual/link4.dae
- added link link4_sc; collision cylinder length=0.12 radius=0.09; collision sphere radius=0.09
- added link link5; collision mesh filename=franka_description/meshes/collision/link5.stl; visual mesh filename=franka_description/meshes/visual/link5.dae
- added link link5_sc; collision cylinder length=0.1 radius=0.09; collision cylinder length=0.14 radius=0.055
- added link link6; collision mesh filename=franka_description/meshes/collision/link6.stl; visual mesh filename=franka_description/meshes/visual/link6.dae
- added link link6_sc; collision cylinder length=0.08 radius=0.08; collision sphere radius=0.08
- added link link7; collision mesh filename=franka_description/meshes/collision/link7.stl; visual mesh filename=franka_description/meshes/visual/link7.dae
- added link link7_sc; collision cylinder length=0.01 radius=0.06; collision cylinder length=0.14 radius=0.07
- added link link8
Joints:
- removed joint panda_joint1
- removed joint panda_joint2
- removed joint panda_joint3
- removed joint panda_joint4
- removed joint panda_joint5
- removed joint panda_joint6
- removed joint panda_joint7
- removed joint panda_joint8
- removed joint panda_link0_sc_joint
- removed joint panda_link1_sc_joint
- removed joint panda_link2_sc_joint
- removed joint panda_link3_sc_joint
- removed joint panda_link4_sc_joint
- removed joint panda_link5_sc_joint
- removed joint panda_link6_sc_joint
- removed joint panda_link7_sc_joint
- added joint joint1: type revolute, parent link0, child link1, origin xyz=0 0 0.333 rpy=0 0 0, axis 0 0 1, limit lower=-2.8973 upper=2.8973 effort=87.0 velocity=2.175
- added joint joint2: type revolute, parent link1, child link2, origin xyz=0 0 0 rpy=-1.5707963267948966 0 0, axis 0 0 1, limit lower=-1.7628 upper=1.7628 effort=87.0 velocity=2.175
- added joint joint3: type revolute, parent link2, child link3, origin xyz=0 -0.316 0 rpy=1.5707963267948966 0 0, axis 0 0 1, limit lower=-2.8973 upper=2.8973 effort=87.0 velocity=2.175
- added joint joint4: type revolute, parent link3, child link4, origin xyz=0.0825 0 0 rpy=1.5707963267948966 0 0, axis 0 0 1, limit lower=-3.0718 upper=-0.0698 effort=87.0 velocity=2.175
- added joint joint5: type revolute, parent link4, child link5, origin xyz=-0.0825 0.384 0 rpy=-1.5707963267948966 0 0, axis 0 0 1, limit lower=-2.8973 upper=2.8973 effort=12.0 velocity=2.61
- added joint joint6: type revolute, parent link5, child link6, origin xyz=0 0 0 rpy=1.5707963267948966 0 0, axis 0 0 1, limit lower=-0.0175 upper=3.7525 effort=12.0 velocity=2.61
- added joint joint7: type revolute, parent link6, child link7, origin xyz=0.088 0 0 rpy=1.5707963267948966 0 0, axis 0 0 1, limit lower=-2.8973 upper=2.8973 effort=12.0 velocity=2.61
- added joint joint8: type fixed, parent link7, child link8, origin xyz=0 0 0.107 rpy=0 0 0
- added joint link0_sc_joint: type fixed, parent link0, child link0_sc, origin rpy=0 0 0
- added joint link1_sc_joint: type fixed, parent link1, child link1_sc, origin rpy=0 0 0
- added joint link2_sc_joint: type fixed, parent link2, child link2_sc, origin rpy=0 0 0
- added joint link3_sc_joint: type fixed, parent link3, child link3_sc, origin rpy=0 0 0
- added joint link4_sc_joint: type fixed, parent link4, child link4_sc, origin rpy=0 0 0
- added joint link5_sc_joint: type fixed, parent link5, child link5_sc, origin rpy=0 0 0
- added joint link6_sc_joint: type fixed, parent link6, child link6_sc, origin rpy=0 0 0
- added joint link7_sc_joint: type fixed, parent link7, child link7_sc, origin rpy=0 0 0.7853981633974483

File: interface/franka_description/panda_arg85.urdf (robot description, URDF)
Before this commit: robot panda, 26 links, 25 joints
Links:
- removed link panda_link0
- removed link panda_link0_sc
- removed link panda_link1
- removed link panda_link1_sc
- removed link panda_link2
- removed link panda_link2_sc
- removed link panda_link3
- removed link panda_link3_sc
- removed link panda_link4
- removed link panda_link4_sc
- removed link panda_link5
- removed link panda_link5_sc
- removed link panda_link6
- removed link panda_link6_sc
- removed link panda_link7
- removed link panda_link7_sc
- removed link panda_link8
- added link link0; collision mesh filename=franka_description/meshes/collision/link0.stl; visual mesh filename=franka_description/meshes/visual/link0.dae
- added link link0_sc; collision cylinder length=0.03 radius=0.09; collision sphere radius=0.09
- added link link1; collision mesh filename=franka_description/meshes/collision/link1.stl; visual mesh filename=franka_description/meshes/visual/link1.dae
- added link link1_sc; collision cylinder length=0.283 radius=0.09; collision sphere radius=0.09
- added link link2; collision mesh filename=franka_description/meshes/collision/link2.stl; visual mesh filename=franka_description/meshes/visual/link2.dae
- added link link2_sc; collision cylinder length=0.12 radius=0.09; collision sphere radius=0.09
- added link link3; collision mesh filename=franka_description/meshes/collision/link3.stl; visual mesh filename=franka_description/meshes/visual/link3.dae
- added link link3_sc; collision cylinder length=0.15 radius=0.09; collision sphere radius=0.09
- added link link4; collision mesh filename=franka_description/meshes/collision/link4.stl; visual mesh filename=franka_description/meshes/visual/link4.dae
- added link link4_sc; collision cylinder length=0.12 radius=0.09; collision sphere radius=0.09
- added link link5; collision mesh filename=franka_description/meshes/collision/link5.stl; visual mesh filename=franka_description/meshes/visual/link5.dae
- added link link5_sc; collision cylinder length=0.1 radius=0.09; collision cylinder length=0.14 radius=0.055
- added link link6; collision mesh filename=franka_description/meshes/collision/link6.stl; visual mesh filename=franka_description/meshes/visual/link6.dae
- added link link6_sc; collision cylinder length=0.08 radius=0.08; collision sphere radius=0.08
- added link link7; collision mesh filename=franka_description/meshes/collision/link7.stl; visual mesh filename=franka_description/meshes/visual/link7.dae
- added link link7_sc; collision cylinder length=0.01 radius=0.06; collision cylinder length=0.14 radius=0.07
- added link link8
Joints:
- removed joint panda_joint1
- removed joint panda_joint2
- removed joint panda_joint3
- removed joint panda_joint4
- removed joint panda_joint5
- removed joint panda_joint6
- removed joint panda_joint7
- removed joint panda_joint8
- removed joint panda_link0_sc_joint
- removed joint panda_link1_sc_joint
- removed joint panda_link2_sc_joint
- removed joint panda_link3_sc_joint
- removed joint panda_link4_sc_joint
- removed joint panda_link5_sc_joint
- removed joint panda_link6_sc_joint
- removed joint panda_link7_sc_joint
- added joint joint1: type revolute, parent link0, child link1, origin xyz=0 0 0.333 rpy=0 0 0, axis 0 0 1, limit lower=-2.8973 upper=2.8973 effort=87.0 velocity=2.175
- added joint joint2: type revolute, parent link1, child link2, origin xyz=0 0 0 rpy=-1.5707963267948966 0 0, axis 0 0 1, limit lower=-1.7628 upper=1.7628 effort=87.0 velocity=2.175
- added joint joint3: type revolute, parent link2, child link3, origin xyz=0 -0.316 0 rpy=1.5707963267948966 0 0, axis 0 0 1, limit lower=-2.8973 upper=2.8973 effort=87.0 velocity=2.175
- added joint joint4: type revolute, parent link3, child link4, origin xyz=0.0825 0 0 rpy=1.5707963267948966 0 0, axis 0 0 1, limit lower=-3.0718 upper=-0.0698 effort=87.0 velocity=2.175
- added joint joint5: type revolute, parent link4, child link5, origin xyz=-0.0825 0.384 0 rpy=-1.5707963267948966 0 0, axis 0 0 1, limit lower=-2.8973 upper=2.8973 effort=12.0 velocity=2.61
- added joint joint6: type revolute, parent link5, child link6, origin xyz=0 0 0 rpy=1.5707963267948966 0 0, axis 0 0 1, limit lower=-0.0175 upper=3.7525 effort=12.0 velocity=2.61
- added joint joint7: type revolute, parent link6, child link7, origin xyz=0.088 0 0 rpy=1.5707963267948966 0 0, axis 0 0 1, limit lower=-2.8973 upper=2.8973 effort=12.0 velocity=2.61
- added joint joint8: type fixed, parent link7, child link8, origin xyz=0 0 0.107 rpy=0 0 0
- added joint link0_sc_joint: type fixed, parent link0, child link0_sc, origin rpy=0 0 0
- added joint link1_sc_joint: type fixed, parent link1, child link1_sc, origin rpy=0 0 0
- added joint link2_sc_joint: type fixed, parent link2, child link2_sc, origin rpy=0 0 0
- added joint link3_sc_joint: type fixed, parent link3, child link3_sc, origin rpy=0 0 0
- added joint link4_sc_joint: type fixed, parent link4, child link4_sc, origin rpy=0 0 0
- added joint link5_sc_joint: type fixed, parent link5, child link5_sc, origin rpy=0 0 0
- added joint link6_sc_joint: type fixed, parent link6, child link6_sc, origin rpy=0 0 0
- added joint link7_sc_joint: type fixed, parent link7, child link7_sc, origin rpy=0 0 0.7853981633974483
- joint robotiq_85_base_joint: parent panda_link8 -> link8

File: interface/franka_description/panda_hande.urdf (robot description, URDF)
Before this commit: robot panda, 21 links, 20 joints
Links:
- removed link panda_link0
- removed link panda_link0_sc
- removed link panda_link1
- removed link panda_link1_sc
- removed link panda_link2
- removed link panda_link2_sc
- removed link panda_link3
- removed link panda_link3_sc
- removed link panda_link4
- removed link panda_link4_sc
- removed link panda_link5
- removed link panda_link5_sc
- removed link panda_link6
- removed link panda_link6_sc
- removed link panda_link7
- removed link panda_link7_sc
- removed link panda_link8
- added link link0; collision mesh filename=franka_description/meshes/collision/link0.stl; visual mesh filename=franka_description/meshes/visual/link0.dae
- added link link0_sc; collision cylinder length=0.03 radius=0.09; collision sphere radius=0.09
- added link link1; collision mesh filename=franka_description/meshes/collision/link1.stl; visual mesh filename=franka_description/meshes/visual/link1.dae
- added link link1_sc; collision cylinder length=0.283 radius=0.09; collision sphere radius=0.09
- added link link2; collision mesh filename=franka_description/meshes/collision/link2.stl; visual mesh filename=franka_description/meshes/visual/link2.dae
- added link link2_sc; collision cylinder length=0.12 radius=0.09; collision sphere radius=0.09
- added link link3; collision mesh filename=franka_description/meshes/collision/link3.stl; visual mesh filename=franka_description/meshes/visual/link3.dae
- added link link3_sc; collision cylinder length=0.15 radius=0.09; collision sphere radius=0.09
- added link link4; collision mesh filename=franka_description/meshes/collision/link4.stl; visual mesh filename=franka_description/meshes/visual/link4.dae
- added link link4_sc; collision cylinder length=0.12 radius=0.09; collision sphere radius=0.09
- added link link5; collision mesh filename=franka_description/meshes/collision/link5.stl; visual mesh filename=franka_description/meshes/visual/link5.dae
- added link link5_sc; collision cylinder length=0.1 radius=0.09; collision cylinder length=0.14 radius=0.055
- added link link6; collision mesh filename=franka_description/meshes/collision/link6.stl; visual mesh filename=franka_description/meshes/visual/link6.dae
- added link link6_sc; collision cylinder length=0.08 radius=0.08; collision sphere radius=0.08
- added link link7; collision mesh filename=franka_description/meshes/collision/link7.stl; visual mesh filename=franka_description/meshes/visual/link7.dae
- added link link7_sc; collision cylinder length=0.01 radius=0.06; collision cylinder length=0.14 radius=0.07
- added link link8
Joints:
- removed joint panda_joint1
- removed joint panda_joint2
- removed joint panda_joint3
- removed joint panda_joint4
- removed joint panda_joint5
- removed joint panda_joint6
- removed joint panda_joint7
- removed joint panda_joint8
- removed joint panda_link0_sc_joint
- removed joint panda_link1_sc_joint
- removed joint panda_link2_sc_joint
- removed joint panda_link3_sc_joint
- removed joint panda_link4_sc_joint
- removed joint panda_link5_sc_joint
- removed joint panda_link6_sc_joint
- removed joint panda_link7_sc_joint
- added joint joint1: type revolute, parent link0, child link1, origin xyz=0 0 0.333 rpy=0 0 0, axis 0 0 1, limit lower=-2.8973 upper=2.8973 effort=87.0 velocity=2.175
- added joint joint2: type revolute, parent link1, child link2, origin xyz=0 0 0 rpy=-1.5707963267948966 0 0, axis 0 0 1, limit lower=-1.7628 upper=1.7628 effort=87.0 velocity=2.175
- added joint joint3: type revolute, parent link2, child link3, origin xyz=0 -0.316 0 rpy=1.5707963267948966 0 0, axis 0 0 1, limit lower=-2.8973 upper=2.8973 effort=87.0 velocity=2.175
- added joint joint4: type revolute, parent link3, child link4, origin xyz=0.0825 0 0 rpy=1.5707963267948966 0 0, axis 0 0 1, limit lower=-3.0718 upper=-0.0698 effort=87.0 velocity=2.175
- added joint joint5: type revolute, parent link4, child link5, origin xyz=-0.0825 0.384 0 rpy=-1.5707963267948966 0 0, axis 0 0 1, limit lower=-2.8973 upper=2.8973 effort=12.0 velocity=2.61
- added joint joint6: type revolute, parent link5, child link6, origin xyz=0 0 0 rpy=1.5707963267948966 0 0, axis 0 0 1, limit lower=-0.0175 upper=3.7525 effort=12.0 velocity=2.61
- added joint joint7: type revolute, parent link6, child link7, origin xyz=0.088 0 0 rpy=1.5707963267948966 0 0, axis 0 0 1, limit lower=-2.8973 upper=2.8973 effort=12.0 velocity=2.61
- added joint joint8: type fixed, parent link7, child link8, origin xyz=0 0 0.107 rpy=0 0 0
- added joint link0_sc_joint: type fixed, parent link0, child link0_sc, origin rpy=0 0 0
- added joint link1_sc_joint: type fixed, parent link1, child link1_sc, origin rpy=0 0 0
- added joint link2_sc_joint: type fixed, parent link2, child link2_sc, origin rpy=0 0 0
- added joint link3_sc_joint: type fixed, parent link3, child link3_sc, origin rpy=0 0 0
- added joint link4_sc_joint: type fixed, parent link4, child link4_sc, origin rpy=0 0 0
- added joint link5_sc_joint: type fixed, parent link5, child link5_sc, origin rpy=0 0 0
- added joint link6_sc_joint: type fixed, parent link6, child link6_sc, origin rpy=0 0 0
- added joint link7_sc_joint: type fixed, parent link7, child link7_sc, origin rpy=0 0 0.7853981633974483
- joint robotiq_hande_coupler: parent panda_link8 -> link8

File: interface/franka_description/panda_hande_d435i.urdf (robot description, URDF)
Before this commit: robot panda, 23 links, 22 joints
Links:
- removed link panda_link0
- removed link panda_link0_sc
- removed link panda_link1
- removed link panda_link1_sc
- removed link panda_link2
- removed link panda_link2_sc
- removed link panda_link3
- removed link panda_link3_sc
- removed link panda_link4
- removed link panda_link4_sc
- removed link panda_link5
- removed link panda_link5_sc
- removed link panda_link6
- removed link panda_link6_sc
- removed link panda_link7
- removed link panda_link7_sc
- removed link panda_link8
- added link link0; collision mesh filename=franka_description/meshes/collision/link0.stl; visual mesh filename=franka_description/meshes/visual/link0.dae
- added link link0_sc; collision cylinder length=0.03 radius=0.09; collision sphere radius=0.09
- added link link1; collision mesh filename=franka_description/meshes/collision/link1.stl; visual mesh filename=franka_description/meshes/visual/link1.dae
- added link link1_sc; collision cylinder length=0.283 radius=0.09; collision sphere radius=0.09
- added link link2; collision mesh filename=franka_description/meshes/collision/link2.stl; visual mesh filename=franka_description/meshes/visual/link2.dae
- added link link2_sc; collision cylinder length=0.12 radius=0.09; collision sphere radius=0.09
- added link link3; collision mesh filename=franka_description/meshes/collision/link3.stl; visual mesh filename=franka_description/meshes/visual/link3.dae
- added link link3_sc; collision cylinder length=0.15 radius=0.09; collision sphere radius=0.09
- added link link4; collision mesh filename=franka_description/meshes/collision/link4.stl; visual mesh filename=franka_description/meshes/visual/link4.dae
- added link link4_sc; collision cylinder length=0.12 radius=0.09; collision sphere radius=0.09
- added link link5; collision mesh filename=franka_description/meshes/collision/link5.stl; visual mesh filename=franka_description/meshes/visual/link5.dae
- added link link5_sc; collision cylinder length=0.1 radius=0.09; collision cylinder length=0.14 radius=0.055
- added link link6; collision mesh filename=franka_description/meshes/collision/link6.stl; visual mesh filename=franka_description/meshes/visual/link6.dae
- added link link6_sc; collision cylinder length=0.08 radius=0.08; collision sphere radius=0.08
- added link link7; collision mesh filename=franka_description/meshes/collision/link7.stl; visual mesh filename=franka_description/meshes/visual/link7.dae
- added link link7_sc; collision cylinder length=0.01 radius=0.06; collision cylinder length=0.14 radius=0.07
- added link link8
Joints:
- removed joint panda_joint1
- removed joint panda_joint2
- removed joint panda_joint3
- removed joint panda_joint4
- removed joint panda_joint5
- removed joint panda_joint6
- removed joint panda_joint7
- removed joint panda_joint8
- removed joint panda_link0_sc_joint
- removed joint panda_link1_sc_joint
- removed joint panda_link2_sc_joint
- removed joint panda_link3_sc_joint
- removed joint panda_link4_sc_joint
- removed joint panda_link5_sc_joint
- removed joint panda_link6_sc_joint
- removed joint panda_link7_sc_joint
- added joint joint1: type revolute, parent link0, child link1, origin xyz=0 0 0.333 rpy=0 0 0, axis 0 0 1, limit lower=-2.8973 upper=2.8973 effort=87.0 velocity=2.175
- added joint joint2: type revolute, parent link1, child link2, origin xyz=0 0 0 rpy=-1.5707963267948966 0 0, axis 0 0 1, limit lower=-1.7628 upper=1.7628 effort=87.0 velocity=2.175
- added joint joint3: type revolute, parent link2, child link3, origin xyz=0 -0.316 0 rpy=1.5707963267948966 0 0, axis 0 0 1, limit lower=-2.8973 upper=2.8973 effort=87.0 velocity=2.175
- added joint joint4: type revolute, parent link3, child link4, origin xyz=0.0825 0 0 rpy=1.5707963267948966 0 0, axis 0 0 1, limit lower=-3.0718 upper=-0.0698 effort=87.0 velocity=2.175
- added joint joint5: type revolute, parent link4, child link5, origin xyz=-0.0825 0.384 0 rpy=-1.5707963267948966 0 0, axis 0 0 1, limit lower=-2.8973 upper=2.8973 effort=12.0 velocity=2.61
- added joint joint6: type revolute, parent link5, child link6, origin xyz=0 0 0 rpy=1.5707963267948966 0 0, axis 0 0 1, limit lower=-0.0175 upper=3.7525 effort=12.0 velocity=2.61
- added joint joint7: type revolute, parent link6, child link7, origin xyz=0.088 0 0 rpy=1.5707963267948966 0 0, axis 0 0 1, limit lower=-2.8973 upper=2.8973 effort=12.0 velocity=2.61
- added joint joint8: type fixed, parent link7, child link8, origin xyz=0 0 0.107 rpy=0 0 0
- added joint link0_sc_joint: type fixed, parent link0, child link0_sc, origin rpy=0 0 0
- added joint link1_sc_joint: type fixed, parent link1, child link1_sc, origin rpy=0 0 0
- added joint link2_sc_joint: type fixed, parent link2, child link2_sc, origin rpy=0 0 0
- added joint link3_sc_joint: type fixed, parent link3, child link3_sc, origin rpy=0 0 0
- added joint link4_sc_joint: type fixed, parent link4, child link4_sc, origin rpy=0 0 0
- added joint link5_sc_joint: type fixed, parent link5, child link5_sc, origin rpy=0 0 0
- added joint link6_sc_joint: type fixed, parent link6, child link6_sc, origin rpy=0 0 0
- added joint link7_sc_joint: type fixed, parent link7, child link7_sc, origin rpy=0 0 0.7853981633974483
- joint d435i_bracket: parent panda_link8 -> link8
